File: Hardware/Qwiic_TMP117.brd (EAGLE design)
At the start: 22.9 x 24.1 mm, 43 parts, among them J1 PTH, U2 TMP117

Commit message: Library created, schematic ready for review, began layout
Parts:
- removed JP10: INT, SparkFun-Passives:PAD-JUMPER-2-NC_BY_TRACE_YES_SILK
- removed JP2, JP3: (no value), SparkFun-Jumpers:SMT-JUMPER_2_NO_SILK
- removed U2: TMP117, TMP117:TMP117
- added U$16: MCP9600-SMD, MCP9600:MQFN-20
- added U$24: CHARLESPAX_TC-MINI-CONNECTOR, MCP9600:CHARLESPAX_TC-MINI-CONNECTOR
- R3: value 10k -> 43k
- moved R3 15.0 mm to (2.54, 16.5), turned to 180 degrees
- moved U$18 14.9 mm to (5.33, 29.2), flipped to the top
- moved U$4 11.6 mm to (13.6, 27.9), flipped to the bottom
- moved U$17 8.98 mm to (20.3, 20.3), turned to 90 degrees
- moved U$2 8.98 mm to (20.3, 20.3), turned to 270 degrees
- moved C1 8.01 mm to (15.4, 11.3), turned to 90 degrees
- moved JP8 6.35 mm to (20.3, 27.9)
- moved JP9 6.35 mm to (2.54, 27.9)
- moved U$6 6.35 mm to (4.06, 25.8)
- moved R2 5.54 mm to (6.22, 16.5)
- moved R4 0.63 mm to (19.1, 5.71)
- moved R5 0.63 mm to (21.6, 5.71)
Connections:
- removed net !INT: J4.1, R3.1, U2.3
- removed net ADD0: JP1.1, JP2.1, JP3.1, R2.1, U2.4
- new net ADDR: JP1.1, R2.1, R3.1, U$16.16
- new net ALT: J4.1, U$16.11
- new net N$7: U$16.4, U$24.P$1
- net 3.3V: now also R3.2, U$16.8; no longer JP10.2, JP3.2, U2.5
- net GND: now also JP1.2, U$16.1, U$16.10, U$16.13, U$16.17, U$16.18, U$16.21, U$16.3, U$16.5, U$16.6, U$16.7, U$16.9; no longer U2.2
- net N$4: now also U$16.2, U$24.P$2; no longer JP10.1, R3.2
- net SCL: now also U$16.19; no longer JP1.2, U2.1
- net SDA: now also U$16.20; no longer JP2.2, U2.6
Routing:
- net 3.3V: track 69.2 -> 0.00 mm, vias 4 -> 0
- net SDA: track 50.8 -> 0.00 mm, vias 3 -> 0
- net SCL: track 47.3 -> 0.00 mm, vias 5 -> 0
- net ADD0: track 18.8 -> 0.00 mm, vias 1 -> 0
- net !INT: track 18.5 -> 0.00 mm
- net GND: track 5.17 -> 0.00 mm, vias 2 -> 0
- net N$2: track 3.70 -> 0.00 mm
- net N$3: track 3.70 -> 0.00 mm
- net N$4: track 3.66 -> 0.00 mm, vias 1 -> 0
- net N$1: track 1.28 -> 0.00 mm
- removed copper zone on layer 16, net N$5
- removed copper zone on layer 1, net N$6
Other:
- board size 22.9 x 24.1 mm -> 22.9 x 30.5 mm
- board text added: "Fischer Moseley"
- board text removed: "Madison Chodikov"
