File: Hardware/Qwiic_TMP117.sch (EAGLE design)
At the start: 21 parts, among them J1 PTH, U2 TMP117

Commit message: Library created, schematic ready for review, began layout
Parts:
- removed JP10: INT, SparkFun-Passives:JUMPER-PAD-2-NC_BY_TRACE
- removed JP2, JP3: JUMPER-SMT_2_NO_SILK, SparkFun-Jumpers:JUMPER-SMT_2_NO_SILK
- removed U2: TMP117, TMP117:TMP117
- added U$16: MCP9600-SMD, MCP9600:MCP9600-SMD
- added U$24: CHARLESPAX_TC-MINI-CONNECTOR, MCP9600:CHARLESPAX_TC-MINI-CONNECTOR
- R3: value 10k -> 43k; device SparkFun-Resistors:10KOHM-0603-1/10W-1% -> SparkFun-Resistors:43KOHM-0603-1/10W-1%
Connections:
- removed net !INT: J4.1, R3.1, U2.!INT
- removed net ADD0: JP1.1, JP2.1, JP3.1, R2.1, U2.ADD0
- new net ADDR: JP1.1, R2.1, R3.1, U$16.ADDR
- new net ALT: J4.1, U$16.ALERT1
- new net N$7: U$16.V-, U$24.P$1
- net 3.3V: now also R3.2, U$16.VDD; no longer JP10.2, JP3.2, U2.V+
- net GND: now also JP1.2, U$16.GND; no longer U2.GND
- net N$4: now also U$16.V+, U$24.P$2; no longer JP10.1, R3.2
- net SCL: now also U$16.SCL; no longer JP1.2, U2.SCL
- net SDA: now also U$16.SDA; no longer JP2.2, U2.SDA
Other:
- note added: "Fischer Moseley"
- note removed: "ADD0 Adress Pin and Slave Adresses GND: 1001000x (0x48) V+: 1001001x (0x49) SDA: 1001010x (0x4A) SCL: 1001011x (0x4B)"
- note removed: "Clear jumper JP10 to remove pull-up from INT"
- note removed: "Madison Chodikov"
- moved on the sheet: I2C, JP1, R2, R3, R4, R5
