File: Hardware/Qwiic_MCP9600.brd (EAGLE design)
At the start: 22.9 x 30.5 mm, 41 parts, among them J1 PTH

Commit message: Push before initial layout review
Parts:
- removed U$1: (no value), buzzard_labels (15):0X4B1
- removed U$18: (no value), buzzard_labels (15):ADR_#_0X484
- removed U$4: (no value), buzzard_labels:TMP1171
- removed U$5: (no value), buzzard_labels (15):0X4A0
- removed U$7: (no value), Labels:INT-()-04
- removed U$8: (no value), buzzard_labels (15):0X493
- added U$25: (no value), MCP9600:MCP96000
- added U$27: (no value), MCP9600:ADR_#_0X600
- moved U$24 34.4 mm to (11.4, 25.9)
- moved R3 15.5 mm to (15.2, 7.62), turned to 0 degrees
- moved JP8 10.2 mm to (20.3, 17.8)
- moved JP9 10.2 mm to (2.54, 17.8)
- moved R2 9.02 mm to (7.75, 7.62), turned to 180 degrees
- moved U$6 8.89 mm to (4.06, 16.9)
- moved JP1 8.80 mm to (11.4, 10.4), turned to 180 degrees
- moved U$17 5.50 mm to (21.0, 25.8)
- moved U$2 5.50 mm to (21.0, 25.8)
- moved R1 0.64 mm to (2.54, 3.17)
- moved I2C 0.51 mm to (20.3, 1.40)
- moved U$21 0.51 mm to (18.4, 3.43)
- moved D1 0.38 mm to (2.54, 4.70)
- moved R4 0.25 mm to (19.1, 5.97)
- moved R5 0.25 mm to (21.6, 5.97)
Other:
- board size 22.9 x 30.5 mm -> 22.9 x 33 mm

Commit message: Push changes made after first layout review
Parts:
- removed U$24: CHARLESPAX_TC-MINI-CONNECTOR, MCP9600:CHARLESPAX_TC-MINI-CONNECTOR
- added JP2: PCB_THERMOCOUPLE, MCP9600:PCC-SMP
- added U$1, U$8: (no value), MCP9600:ART10
- added U$18, U$5: (no value), MCP9600:ART40
- added U$4: (no value), MCP9600:ART30
- added U$7: (no value), MCP9600:ART20
- J4: device SparkFun-Connectors:1X01_NO_SILK -> SparkFun-Connectors:1X04_NO_SILK
- R2: value 10k -> 43k
- R3: value 43k -> 10k
- U$11: device Labels:INT#-[<-04 -> MCP9600:ART30
- U$3: device Labels:INT#-[<-04 -> MCP9600:ART20
- moved U$15 38.1 mm to (36.3, 27.3)
- moved U$21 16.2 mm to (14.0, 19.1)
- moved I2C 15.9 mm to (15.9, 16.6)
- moved U$25 15.2 mm to (7.24, 30.4)
- moved U$6 15.2 mm to (4.06, 32.1)
- moved R4 15.0 mm to (4.19, 7.62), turned to 0 degrees
- moved LOGO1 13.7 mm to (7.62, 16.5)
- moved R1 13.7 mm to (7.62, 15.9), turned to 180 degrees
- moved D1 13.6 mm to (7.62, 17.3), turned to 0 degrees
- moved U$20 13.4 mm to (4.95, 19.1)
- moved R5 13.3 mm to (8.38, 7.62), turned to 0 degrees
- moved U$17 9.53 mm to (11.4, 25.9), turned to 0 degrees
- moved U$2 9.53 mm to (11.4, 25.9), turned to 0 degrees
- moved C1 7.88 mm to (7.49, 10.9), turned to 270 degrees
- moved R3 6.66 mm to (11.4, 2.16), turned to 270 degrees
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Connections:
- net ALT renamed ALRT1
- removed net N$7: U$16.4, U$24.P$1
- new net ALRT2: J4.2, U$16.12
- new net ALRT3: J4.3, U$16.14
- new net ALRT4: J4.4, U$16.15
- new net N$5: JP2.-, U$16.4
- net N$4: now also JP2.+; no longer U$24.P$2
Routing:
- net 3.3V: track 0.00 -> 57.4 mm, vias 0 -> 2
- net GND: track 0.00 -> 41.1 mm
- net SDA: track 0.00 -> 30.4 mm, vias 0 -> 2
- net SCL: track 0.00 -> 27.9 mm, vias 0 -> 2
- net ADDR: track 0.00 -> 17.2 mm, vias 0 -> 2
- net N$3: track 0.00 -> 16.3 mm, vias 0 -> 2
- net N$2: track 0.00 -> 15.4 mm, vias 0 -> 2
- net ALRT4: track 0.00 -> 12.5 mm
- net ALRT3: track 0.00 -> 11.4 mm
- net ALRT2: track 0.00 -> 10.9 mm
- net N$5: track 0.00 -> 10.9 mm
- net N$4: track 0.00 -> 10.9 mm
- net ALRT1: track 0.00 -> 10.1 mm
- net N$1: track 0.00 -> 1.41 mm
Other:
- board size 22.9 x 33 mm -> 22.9 x 36.8 mm

Commit message: Changed MCP9600 designator
U$16 -> U16
Parts:
- renumbered U$16 to U16
Changed lines of the file:
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@@
 <drawing>
 <settings>
-<setting alwaysvectorfont="yes"/>
+<setting alwaysvectorfont="no"/>
 <setting verticaltext="up"/>
 </settings>
@@
 <element name="U$14" library="Labels" package="SDA-[)" value="" x="6.35" y="1.651" smashed="yes" rot="MR90"/>
 <element name="U$15" library="SparkFun-Aesthetics" package="QWIIC_5.5MM" value="" x="36.322" y="27.305" smashed="yes" rot="MR0"/>
-<element name="U$16" library="MCP9600" package="MQFN-20" value="MCP9600-SMD" x="11.43" y="12.065" smashed="yes" rot="R270"/>
+<element name="U16" library="MCP9600" package="MQFN-20" value="MCP9600-SMD" x="11.43" y="12.065" smashed="yes" rot="R270"/>
 <element name="R3" library="SparkFun-Resistors" package="0603" value="10k" x="11.43" y="2.159" smashed="yes" rot="R270">
 <attribute name="PROD_ID" value="RES-00824" x="11.43" y="2.159" size="1.778" layer="27" rot="R270" display="off"/>
@@
 <vertex x="22.86" y="0"/>
 </polygon>
-<contactref element="U$16" pad="1"/>
-<contactref element="U$16" pad="17"/>
-<contactref element="U$16" pad="6"/>
-<contactref element="U$16" pad="9"/>
-<contactref element="U$16" pad="3"/>
-<contactref element="U$16" pad="5"/>
-<contactref element="U$16" pad="21"/>
-<contactref element="U$16" pad="7"/>
-<contactref element="U$16" pad="13"/>
-<contactref element="U$16" pad="18"/>
-<contactref element="U$16" pad="10"/>
+<contactref element="U16" pad="1"/>
+<contactref element="U16" pad="17"/>
+<contactref element="U16" pad="6"/>
+<contactref element="U16" pad="9"/>
+<contactref element="U16" pad="3"/>
+<contactref element="U16" pad="5"/>
+<contactref element="U16" pad="21"/>
+<contactref element="U16" pad="7"/>
+<contactref element="U16" pad="13"/>
+<contactref element="U16" pad="18"/>
+<contactref element="U16" pad="10"/>
 <contactref element="JP1" pad="2"/>
 <wire x1="9.18" y1="13.365" x2="8.98" y2="13.565" width="0.1778" layer="1"/>
@@
 <contactref element="J2" pad="2"/>
 <contactref element="I2C" pad="2"/>
-<contactref element="U$16" pad="8"/>
+<contactref element="U16" pad="8"/>
 <contactref element="R3" pad="2"/>
 <wire x1="9.18" y1="12.065" x2="7.786" y2="12.065" width="0.1778" layer="1"/>
@@
 <contactref element="J3" pad="3"/>
 <contactref element="R4" pad="1"/>
-<contactref element="U$16" pad="20"/>
+<contactref element="U16" pad="20"/>
 <wire x1="18.7217" y1="13.97546875" x2="18.7217" y2="13.15453125" width="0.1778" layer="1"/>
 <wire x1="18.7217" y1="13.15453125" x2="17.91156875" y2="12.3444" width="0.1778" layer="1"/>
@@
 <contactref element="JP1" pad="1"/>
 <contactref element="R2" pad="1"/>
-<contactref element="U$16" pad="16"/>
+<contactref element="U16" pad="16"/>
 <contactref element="R3" pad="1"/>
 <wire x1="11.43" y1="3.009" x2="11.43" y2="4.738" width="0.1778" layer="1"/>
@@
 <contactref element="J1" pad="4"/>
 <contactref element="R5" pad="1"/>
-<contactref element="U$16" pad="19"/>
+<contactref element="U16" pad="19"/>
 <wire x1="13.68" y1="12.715" x2="13.695" y2="12.7" width="0.1778" layer="1"/>
 <wire x1="7.532" y1="7.62" x2="7.517" y2="7.62" width="0.1778" layer="1"/>
@@
 </signal>
 <signal name="N$4">
-<contactref element="U$16" pad="2"/>
+<contactref element="U16" pad="2"/>
 <contactref element="JP2" pad="+"/>
 <wire x1="12.08" y1="14.315" x2="12.08" y2="17.16" width="0.1778" layer="1"/>
@@
 </signal>
 <signal name="N$5">
-<contactref element="U$16" pad="4"/>
+<contactref element="U16" pad="4"/>
 <contactref element="JP2" pad="-"/>
 <wire x1="10.78" y1="14.315" x2="10.78" y2="17.16" width="0.1778" layer="1"/>
@@
 </signal>
 <signal name="ALRT1">
-<contactref element="U$16" pad="11"/>
+<contactref element="U16" pad="11"/>
 <contactref element="J4" pad="1"/>
 <wire x1="13.97" y1="1.27" x2="13.97" y2="5.715" width="0.1778" layer="1"/>
@@
 </signal>
 <signal name="ALRT2">
-<contactref element="U$16" pad="12"/>
+<contactref element="U16" pad="12"/>
 <contactref element="J4" pad="2"/>
 <wire x1="16.51" y1="1.27" x2="16.51" y2="3.88283125" width="0.1778" layer="1"/>
@@
 </signal>
 <signal name="ALRT3">
-<contactref element="U$16" pad="14"/>
+<contactref element="U16" pad="14"/>
 <contactref element="J4" pad="3"/>
 <wire x1="12.08" y1="9.815" x2="12.08" y2="9.51" width="0.1778" layer="1"/>
@@
 </signal>
 <signal name="ALRT4">
-<contactref element="U$16" pad="15"/>
+<contactref element="U16" pad="15"/>
 <contactref element="J4" pad="4"/>
 <wire x1="21.082" y1="1.27" x2="12.73" y2="9.622" width="0.1778" layer="1"/>
