File: Hardware/Qwiic_MCP9600.sch (EAGLE design)
At the start: 19 parts, among them J1 PTH

Commit message: Push before initial layout review
Other:
- note added: "MCP9600 Thermocouple EMF to Temperature Converter"
- note removed: "TMP117 Temperature Sensor"
Changed lines of the file:
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@@
 <wire x1="0" y1="96.52" x2="248.92" y2="96.52" width="0.1524" layer="97" style="longdash"/>
 <text x="45.72" y="86.36" size="1.778" layer="97" font="vector">I2C Connections</text>
-<text x="88.9" y="177.8" size="1.778" layer="97" font="vector">TMP117 Temperature Sensor</text>
+<text x="88.9" y="177.8" size="1.778" layer="97" font="vector">MCP9600 Thermocouple EMF to Temperature Converter</text>
 <text x="167.894" y="11.43" size="2.54" layer="94" font="vector">Fischer Moseley</text>
 <text x="137.16" y="167.64" size="1.778" layer="97" font="vector" rot="MR0">Clear Jumper to remove

Commit message: Push changes made after first layout review
Parts:
- removed U$24: CHARLESPAX_TC-MINI-CONNECTOR, MCP9600:CHARLESPAX_TC-MINI-CONNECTOR
- added JP2: PCB_THERMOCOUPLE, MCP9600:PCB_THERMOCOUPLE
- J4: device SparkFun-Connectors:CONN_01PTH_NO_SILK_YES_STOP -> SparkFun-Connectors:CONN_041X04_NO_SILK
- R2: value 10k -> 43k; device SparkFun-Resistors:10KOHM-0603-1/10W-1% -> SparkFun-Resistors:43KOHM-0603-1/10W-1%
- R3: value 43k -> 10k; device SparkFun-Resistors:43KOHM-0603-1/10W-1% -> SparkFun-Resistors:10KOHM-0603-1/10W-1%
Connections:
- net ALT renamed ALRT1
- removed net N$7: U$16.V-, U$24.P$1
- new net ALRT2: J4.2, U$16.ALERT2
- new net ALRT3: J4.3, U$16.ALERT3
- new net ALRT4: J4.4, U$16.ALERT4
- new net N$5: JP2G$1.-, U$16.V-
- net N$4: now also JP2G$1.+; no longer U$24.P$2
Other:
- moved on the sheet: I2C, JP1, R2, R3, R4, R5

Commit message: Changed MCP9600 designator
U$16 -> U16
Parts:
- renumbered U$16 to U16
Changed lines of the file:
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@@
 <part name="JP9" library="SparkFun" deviceset="STAND-OFF" device=""/>
 <part name="I2C" library="SparkFun-Jumpers" deviceset="JUMPER-SMT_3_2-NC_TRACE" device="_SILK" value=""/>
-<part name="U$16" library="MCP9600" deviceset="MCP9600" device="-SMD"/>
+<part name="U16" library="MCP9600" deviceset="MCP9600" device="-SMD"/>
 <part name="R3" library="SparkFun-Resistors" deviceset="10KOHM" device="-0603-1/10W-1%" value="10k"/>
 <part name="SUPPLY2" library="SparkFun-PowerSymbols" library_urn="urn:adsk.eagle:library:530" deviceset="3.3V" device=""/>
@@
 <attribute name="VALUE" x="157.861" y="152.4" size="1.778" layer="96" font="vector" rot="MR270" align="top-left"/>
 </instance>
-<instance part="U$16" gate="G$1" x="190.5" y="137.16" smashed="yes">
+<instance part="U16" gate="G$1" x="190.5" y="137.16" smashed="yes">
 <attribute name="NAME" x="180.34" y="124.46" size="1.778" layer="95"/>
 <attribute name="VALUE" x="180.34" y="148.082" size="1.778" layer="96"/>
@@
 <wire x1="175.26" y1="127" x2="175.26" y2="129.54" width="0.1524" layer="91"/>
 <wire x1="175.26" y1="129.54" x2="177.8" y2="129.54" width="0.1524" layer="91"/>
-<pinref part="U$16" gate="G$1" pin="GND"/>
+<pinref part="U16" gate="G$1" pin="GND"/>
 </segment>
 <segment>
@@
 <wire x1="175.26" y1="147.32" x2="175.26" y2="144.78" width="0.1524" layer="91"/>
 <wire x1="175.26" y1="144.78" x2="177.8" y2="144.78" width="0.1524" layer="91"/>
-<pinref part="U$16" gate="G$1" pin="VDD"/>
+<pinref part="U16" gate="G$1" pin="VDD"/>
 </segment>
 <segment>
@@
 <junction x="165.1" y="139.7"/>
 <label x="144.78" y="139.7" size="1.27" layer="95" rot="MR0" xref="yes"/>
-<pinref part="U$16" gate="G$1" pin="SDA"/>
+<pinref part="U16" gate="G$1" pin="SDA"/>
 <wire x1="165.1" y1="139.7" x2="177.8" y2="139.7" width="0.1524" layer="91"/>
 </segment>
@@
 <junction x="149.86" y="137.16"/>
 <label x="144.78" y="137.16" size="1.27" layer="95" rot="MR0" xref="yes"/>
-<pinref part="U$16" gate="G$1" pin="SCL"/>
+<pinref part="U16" gate="G$1" pin="SCL"/>
 </segment>
 </net>
@@
 <junction x="124.46" y="134.62"/>
 <label x="121.92" y="134.62" size="1.27" layer="95" rot="MR0" xref="yes"/>
-<pinref part="U$16" gate="G$1" pin="ADDR"/>
+<pinref part="U16" gate="G$1" pin="ADDR"/>
 <wire x1="137.16" y1="134.62" x2="177.8" y2="134.62" width="0.1524" layer="91"/>
 <pinref part="R3" gate="G$1" pin="1"/>
@@
 <net name="N$4" class="0">
 <segment>
-<pinref part="U$16" gate="G$1" pin="V+"/>
+<pinref part="U16" gate="G$1" pin="V+"/>
 <pinref part="JP2" gate="G$1" pin="+"/>
 <wire x1="203.2" y1="144.78" x2="218.44" y2="144.78" width="0.1524" layer="91"/>
@@
 <net name="N$5" class="0">
 <segment>
-<pinref part="U$16" gate="G$1" pin="V-"/>
+<pinref part="U16" gate="G$1" pin="V-"/>
 <pinref part="JP2" gate="G$1" pin="-"/>
 <wire x1="203.2" y1="142.24" x2="218.44" y2="142.24" width="0.1524" layer="91"/>
@@
 <net name="ALRT1" class="0">
 <segment>
-<pinref part="U$16" gate="G$1" pin="ALERT1"/>
+<pinref part="U16" gate="G$1" pin="ALERT1"/>
 <wire x1="203.2" y1="137.16" x2="208.28" y2="137.16" width="0.1524" layer="91"/>
 <label x="208.28" y="137.16" size="1.27" layer="95" xref="yes"/>
@@
 <net name="ALRT2" class="0">
 <segment>
-<pinref part="U$16" gate="G$1" pin="ALERT2"/>
+<pinref part="U16" gate="G$1" pin="ALERT2"/>
 <wire x1="203.2" y1="134.62" x2="208.28" y2="134.62" width="0.1524" layer="91"/>
 <label x="208.28" y="134.62" size="1.27" layer="95" xref="yes"/>
@@
 <net name="ALRT3" class="0">
 <segment>
-<pinref part="U$16" gate="G$1" pin="ALERT3"/>
+<pinref part="U16" gate="G$1" pin="ALERT3"/>
 <wire x1="203.2" y1="132.08" x2="208.28" y2="132.08" width="0.1524" layer="91"/>
 <label x="208.28" y="132.08" size="1.27" layer="95" xref="yes"/>
@@
 <net name="ALRT4" class="0">
 <segment>
-<pinref part="U$16" gate="G$1" pin="ALERT4"/>
+<pinref part="U16" gate="G$1" pin="ALERT4"/>
 <wire x1="203.2" y1="129.54" x2="208.28" y2="129.54" width="0.1524" layer="91"/>
 <label x="208.28" y="129.54" size="1.27" layer="95" xref="yes"/>

Commit message: Added addressing information to schematic
Other:
- note added: "MCP9600 Address Selection: 0x60: ADDR tied to GND 0x61: R3 = 10k, R2 = 2.2k 0x62: R3 = 10k, R2 = 4.3k 0x63: R3 = 10k, R2 = 7.5k 0x64: R3 = 10k, R2 = 13k 0x65: R3 = 10k, R2 = 22k 0x66: R3 = 10k, R2 = 43k 0x66: ADDR Pin Tied to VDD"
Changed lines of the file:
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@@
 <text x="149.86" y="167.64" size="1.778" layer="97" font="vector" rot="MR0">Clear Jumper to remove
 I2C Pull-ups from bus</text>
+<text x="76.2" y="114.3" size="1.524" layer="97" font="vector">MCP9600 Address Selection:
+0x60: ADDR tied to GND
+0x61: R3 = 10k, R2 = 2.2k
+0x62: R3 = 10k, R2 = 4.3k
+0x63: R3 = 10k, R2 = 7.5k
+0x64: R3 = 10k, R2 = 13k
+0x65: R3 = 10k, R2 = 22k
+0x66: R3 = 10k, R2 = 43k
+0x66: ADDR Pin Tied to VDD </text>
 </plain>
 <instances>

Commit message: Added production files
Connections:
- net ALRT1 renamed !ALT1
- net ALRT2 renamed !ALT2
- net ALRT3 renamed !ALT3
- net ALRT4 renamed !ALT4
Other:
- note added: "Clear jumper to remove I2C pullups"
- note added: "MCP9600 Address Selection: 0x60: ADDR tied to GND 0x61: R3 = 10k, R2 = 2.2k 0x62: R3 = 10k, R2 = 4.3k 0x63: R3 = 10k, R2 = 7.5k 0x64: R3 = 10k, R2 = 13k 0x65: R3 = 10k, R2 = 22k 0x66: R3 = 10k, R2 = 43k (default) 0x66: ADDR Pin Tied to VDD"
- note added: "x01"
- note removed: "Clear Jumper to remove I2C Pull-ups from bus"
- note removed: "MCP9600 Address Selection: 0x60: ADDR tied to GND 0x61: R3 = 10k, R2 = 2.2k 0x62: R3 = 10k, R2 = 4.3k 0x63: R3 = 10k, R2 = 7.5k 0x64: R3 = 10k, R2 = 13k 0x65: R3 = 10k, R2 = 22k 0x66: R3 = 10k, R2 = 43k 0x66: ADDR Pin Tied to VDD"
Changed lines of the file:
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@@
 <drawing>
 <settings>
-<setting alwaysvectorfont="no"/>
+<setting alwaysvectorfont="yes"/>
 <setting verticaltext="up"/>
 </settings>
@@
 <text x="88.9" y="177.8" size="1.778" layer="97" font="vector">MCP9600 Thermocouple EMF to Temperature Converter</text>
 <text x="167.894" y="11.43" size="2.54" layer="94" font="vector">Fischer Moseley</text>
-<text x="149.86" y="167.64" size="1.778" layer="97" font="vector" rot="MR0">Clear Jumper to remove
-I2C Pull-ups from bus</text>
+<text x="149.86" y="167.64" size="1.778" layer="97" font="vector" rot="MR0">Clear jumper to remove
+I2C pullups</text>
 <text x="76.2" y="114.3" size="1.524" layer="97" font="vector">MCP9600 Address Selection:
 0x60: ADDR tied to GND
@@
 0x64: R3 = 10k, R2 = 13k
 0x65: R3 = 10k, R2 = 22k
-0x66: R3 = 10k, R2 = 43k
+0x66: R3 = 10k, R2 = 43k (default)
 0x66: ADDR Pin Tied to VDD </text>
+<text x="239.522" y="7.366" size="2.54" layer="94">x01</text>
 </plain>
 <instances>
@@
 </instance>
 <instance part="U16" gate="G$1" x="190.5" y="137.16" smashed="yes">
-<attribute name="NAME" x="180.34" y="124.46" size="1.778" layer="95"/>
-<attribute name="VALUE" x="180.34" y="148.082" size="1.778" layer="96"/>
+<attribute name="NAME" x="180.34" y="124.46" size="1.778" layer="95" font="vector"/>
+<attribute name="VALUE" x="180.34" y="148.082" size="1.778" layer="96" font="vector"/>
 </instance>
 <instance part="R3" gate="G$1" x="124.46" y="142.24" smashed="yes" rot="R90">
@@
 <pinref part="JP1" gate="G$1" pin="1"/>
 <wire x1="137.16" y1="132.08" x2="137.16" y2="134.62" width="0.1524" layer="91"/>
-<junction x="137.16" y="134.62"/>
 <pinref part="R2" gate="G$1" pin="1"/>
 <wire x1="137.16" y1="134.62" x2="124.46" y2="134.62" width="0.1524" layer="91"/>
@@
 <junction x="124.46" y="134.62"/>
 <label x="121.92" y="134.62" size="1.27" layer="95" rot="MR0" xref="yes"/>
+<pinref part="R3" gate="G$1" pin="1"/>
+<wire x1="124.46" y1="137.16" x2="124.46" y2="134.62" width="0.1524" layer="91"/>
 <pinref part="U16" gate="G$1" pin="ADDR"/>
 <wire x1="137.16" y1="134.62" x2="177.8" y2="134.62" width="0.1524" layer="91"/>
-<pinref part="R3" gate="G$1" pin="1"/>
-<wire x1="124.46" y1="137.16" x2="124.46" y2="134.62" width="0.1524" layer="91"/>
+<junction x="137.16" y="134.62"/>
 </segment>
 </net>
@@
 </segment>
 </net>
-<net name="N$8" class="0">
-<segment>
-<wire x1="154.94" y1="134.62" x2="152.4" y2="134.62" width="0.1524" layer="91"/>
-</segment>
-</net>
 <net name="N$4" class="0">
 <segment>
@@
 </segment>
 </net>
-<net name="ALRT1" class="0">
+<net name="!ALT1" class="0">
+<segment>
+<wire x1="68.58" y1="40.64" x2="66.04" y2="40.64" width="0.1524" layer="91"/>
+<label x="66.04" y="40.64" size="1.27" layer="95" rot="R180" xref="yes"/>
+<pinref part="J4" gate="J1" pin="1"/>
+</segment>
 <segment>
 <pinref part="U16" gate="G$1" pin="ALERT1"/>
@@
 <label x="208.28" y="137.16" size="1.27" layer="95" xref="yes"/>
 </segment>
-<segment>
-<wire x1="68.58" y1="40.64" x2="66.04" y2="40.64" width="0.1524" layer="91"/>
-<label x="66.04" y="40.64" size="1.27" layer="95" rot="R180" xref="yes"/>
-<pinref part="J4" gate="J1" pin="1"/>
-</segment>
-</net>
-<net name="ALRT2" class="0">
+</net>
+<net name="!ALT3" class="0">
+<segment>
+<wire x1="68.58" y1="35.56" x2="66.04" y2="35.56" width="0.1524" layer="91"/>
+<label x="66.04" y="35.56" size="1.27" layer="95" rot="R180" xref="yes"/>
+<pinref part="J4" gate="J1" pin="3"/>
+</segment>
+<segment>
+<pinref part="U16" gate="G$1" pin="ALERT3"/>
+<wire x1="203.2" y1="132.08" x2="208.28" y2="132.08" width="0.1524" layer="91"/>
+<label x="208.28" y="132.08" size="1.27" layer="95" xref="yes"/>
+</segment>
+</net>
+<net name="!ALT4" class="0">
+<segment>
+<wire x1="68.58" y1="33.02" x2="66.04" y2="33.02" width="0.1524" layer="91"/>
+<label x="66.04" y="33.02" size="1.27" layer="95" rot="R180" xref="yes"/>
+<pinref part="J4" gate="J1" pin="4"/>
+</segment>
+<segment>
+<pinref part="U16" gate="G$1" pin="ALERT4"/>
+<wire x1="203.2" y1="129.54" x2="208.28" y2="129.54" width="0.1524" layer="91"/>
+<label x="208.28" y="129.54" size="1.27" layer="95" xref="yes"/>
+</segment>
+</net>
+<net name="!ALT2" class="0">
+<segment>
+<wire x1="68.58" y1="38.1" x2="66.04" y2="38.1" width="0.1524" layer="91"/>
+<label x="66.04" y="38.1" size="1.27" layer="95" rot="R180" xref="yes"/>
+<pinref part="J4" gate="J1" pin="2"/>
+</segment>
 <segment>
 <pinref part="U16" gate="G$1" pin="ALERT2"/>
@@
 <label x="208.28" y="134.62" size="1.27" layer="95" xref="yes"/>
 </segment>
-<segment>
-<wire x1="68.58" y1="38.1" x2="66.04" y2="38.1" width="0.1524" layer="91"/>
-<label x="66.04" y="38.1" size="1.27" layer="95" rot="R180" xref="yes"/>
-<pinref part="J4" gate="J1" pin="2"/>
-</segment>
-</net>
-<net name="ALRT3" class="0">
-<segment>
-<pinref part="U16" gate="G$1" pin="ALERT3"/>
-<wire x1="203.2" y1="132.08" x2="208.28" y2="132.08" width="0.1524" layer="91"/>
-<label x="208.28" y="132.08" size="1.27" layer="95" xref="yes"/>
-</segment>
-<segment>
-<wire x1="68.58" y1="35.56" x2="66.04" y2="35.56" width="0.1524" layer="91"/>
-<label x="66.04" y="35.56" size="1.27" layer="95" rot="R180" xref="yes"/>
-<pinref part="J4" gate="J1" pin="3"/>
-</segment>
-</net>
-<net name="ALRT4" class="0">
-<segment>
-<pinref part="U16" gate="G$1" pin="ALERT4"/>
-<wire x1="203.2" y1="129.54" x2="208.28" y2="129.54" width="0.1524" layer="91"/>
-<label x="208.28" y="129.54" size="1.27" layer="95" xref="yes"/>
-</segment>
-<segment>
-<wire x1="68.58" y1="33.02" x2="66.04" y2="33.02" width="0.1524" layer="91"/>
-<label x="66.04" y="33.02" size="1.27" layer="95" rot="R180" xref="yes"/>
-<pinref part="J4" gate="J1" pin="4"/>
-</segment>
-</net>
+</net>
